Commit message: [WIP] moveit

File: motoman_description/robots/hc10.xacro (robot description, xacro)
@@ -3,7 +3,16 @@
   <xacro:arg name="arm_id" default=""/> <!-- Name of this robot, not used yet -->
   <xacro:arg name="robot_ip" default=""/> <!-- IP address or hostname of the robot" -->
+  <xacro:arg name="use_mock_hardware" default="false"/> <!-- Mirror commands to hardware states -->
+  <xacro:arg name="mock_sensor_commands" default="false"/> <!-- Use fake sensor input-->
+  <xacro:arg name="sim_gazebo" default="false" /> <!-- Use gazebo simulation-->
   <xacro:include filename="$(find motoman_description)/robots/hc10_macro.xacro" />
   <xacro:motoman_hc10 prefix=""/>
   <xacro:include filename="$(find motoman_description)/robots/ros2_control.xacro"/>
-  <xacro:motoman_ros2_control ns="$(arg arm_id)" robot_ip="$(arg robot_ip)"/>
+  <xacro:motoman_ros2_control
+    ns="$(arg arm_id)"
+    robot_ip="$(arg robot_ip)"
+    use_mock_hardware="$(arg use_mock_hardware)"
+    mock_sensor_commands="$(arg mock_sensor_commands)"
+    sim_gazebo="$(arg sim_gazebo)"
+  />
 </robot>

File: motoman_description/robots/ros2_control.xacro (robot description, xacro)
@@ -1,12 +1,23 @@
-<?xml version="1.0" ?>
+<?xml version="1.0"?>
 <robot xmlns:xacro="http://www.ros.org/wiki/xacro">
-    <xacro:macro name="motoman_ros2_control" params="ns robot_ip">
+    <xacro:macro name="motoman_ros2_control" params="
+            ns
+            robot_ip
+            use_mock_hardware:=^|false
+            mock_sensor_commands:=^|false
+            sim_gazebo:=^|false
+            ">
         <ros2_control name="MotomanHardware" type="system">
+            <!-- THIS IS JUST FOR REFERENCE! -->
             <!-- <xacro:macro name="configure_joint" params="joint_name initial_position">
                 <joint name="${joint_name}">
                 <param name="initial_position">${initial_position}</param>
                     <command_interface name="position"/>
-                    <state_interface name="position"/>
-                    <state_interface name="velocity"/>
+                    <state_interface name="position">
+                        <param name="initial_value">0.0</param>
+                    </state_interface>
+                    <state_interface name="velocity">
+                        <param name="initial_value">0.0</param>
+                    </state_interface>
                     <state_interface name="effort"/>
                 </joint>
@@ -14,58 +25,88 @@
             <xacro:configure_joint joint_name="${ns}_joint1" initial_position="0.0"/> -->
             <hardware>
-                <plugin>motoman_hardware/MotomanHardware</plugin>
+                <xacro:if value="${use_mock_hardware}">
+                    <plugin>mock_components/GenericSystem</plugin>
+                    <param name="mock_sensor_commands">${mock_sensor_commands}</param>
+                </xacro:if>
+                <xacro:unless value="${use_mock_hardware or sim_gazebo}">
+                    <plugin>motoman_hardware/MotomanHardware</plugin>
+                    <param name="udp_ip_address">${robot_ip}</param>
+                    <param name="udp_port">50244</param>
+                </xacro:unless>
                 <!-- <param name="example_param_hw_start_duration_sec">2.0</param>
                 <param name="example_param_hw_stop_duration_sec">3.0</param>
                 <param name="example_param_hw_slowdown">2.0</param> -->
-                <param name="udp_ip_address">${robot_ip}</param>
-                <param name="udp_port">50244</param>
             </hardware>
             <joint name="joint_1_s">
                 <command_interface name="position">
-                <param name="min">-1</param>
-                <param name="max">1</param>
+                <!-- <param name="min">-1</param> -->
+                <!-- <param name="max">1</param> -->
                 </command_interface>
-                <state_interface name="position"/>
-                <state_interface name="velocity"/>
+                <state_interface name="position">
+                    <param name="initial_value">0.0</param>
+                </state_interface>
+                <state_interface name="velocity">
+                    <param name="initial_value">0.0</param>
+                </state_interface>
             </joint>
             <joint name="joint_2_l">
                 <command_interface name="position">
-                <param name="min">-1</param>
-                <param name="max">1</param>
+                <!-- <param name="min">-1</param> -->
+                <!-- <param name="max">1</param> -->
                 </command_interface>
-                <state_interface name="position"/>
-                <state_interface name="velocity"/>
+                <state_interface name="position">
+                    <param name="initial_value">0.0</param>
+                </state_interface>
+                <state_interface name="velocity">
+                    <param name="initial_value">0.0</param>
+                </state_interface>
             </joint>
             <joint name="joint_3_u">
                 <command_interface name="position">
-                <param name="min">-1</param>
-                <param name="max">1</param>
+                <!-- <param name="min">-1</param> -->
+                <!-- <param name="max">1</param> -->
                 </command_interface>
-                <state_interface name="position"/>
-                <state_interface name="velocity"/>
+                <state_interface name="position">
+                    <param name="initial_value">0.7</param>
+                </state_interface>
+                <state_interface name="velocity">
+                    <param name="initial_value">0.0</param>
+                </state_interface>
             </joint>
             <joint name="joint_4_r">
                 <command_interface name="position">
-                <param name="min">-1</param>
-                <param name="max">1</param>
+                <!-- <param name="min">-1</param> -->
+                <!-- <param name="max">1</param> -->
                 </command_interface>
-                <state_interface name="position"/>
-                <state_interface name="velocity"/>
+                <state_interface name="position">
+                    <param name="initial_value">0.7</param>
+                </state_interface>
+                <state_interface name="velocity">
+                    <param name="initial_value">0.0</param>
+                </state_interface>
             </joint>
             <joint name="joint_5_b">
                 <command_interface name="position">
-                <param name="min">-1</param>
-                <param name="max">1</param>
+                <!-- <param name="min">-1</param> -->
+                <!-- <param name="max">1</param> -->
                 </command_interface>
-                <state_interface name="position"/>
-                <state_interface name="velocity"/>
+                <state_interface name="position">
+                    <param name="initial_value">0.7</param>
+                </state_interface>
+                <state_interface name="velocity">
+                    <param name="initial_value">0.0</param>
+                </state_interface>
             </joint>
             <joint name="joint_6_t">
                 <command_interface name="position">
-                <param name="min">-1</param>
-                <param name="max">1</param>
+                <!-- <param name="min">-1</param> -->
+                <!-- <param name="max">1</param> -->
                 </command_interface>
-                <state_interface name="position"/>
-                <state_interface name="velocity"/>
+                <state_interface name="position">
+                    <param name="initial_value">0.0</param>
+                </state_interface>
+                <state_interface name="velocity">
+                    <param name="initial_value">0.0</param>
+                </state_interface>
             </joint>
         </ros2_control>
