Commit message: [WIP] latency tests fix 1

File: motoman_description/robots/hc10_macro.xacro (robot description, xacro)
@@ -146,4 +146,11 @@
     </joint>
     <!-- end of joint list -->
+    <!-- robot tracking target -->
+    <link name="${prefix}tool_marker"/>
+    <joint name="${prefix}tool0-marker" type="fixed">
+      <origin xyz="0 0 0.1" rpy="0 0 0"/>
+      <parent link="${prefix}tool0"/>
+      <child link="${prefix}tool_marker"/>
+    </joint>
     <!-- ROS base_link to Robot Manufacturer World Coordinates transform -->
     <link name="${prefix}base" />
@@ -153,4 +160,11 @@
       <child link="${prefix}base"/>
     </joint>
+    <!-- create link fixed to the "world" -->
+    <link name="world" />
+    <joint name="${prefix}world-base_link" type="fixed">
+      <origin xyz="0 0 0" rpy="0 0 0"/>
+      <parent link="${prefix}world"/>
+      <child link="${prefix}base_link"/>
+    </joint>
   </xacro:macro>
 </robot>

File: motoman_description/robots/ros2_control.xacro (robot description, xacro)
@@ -21,4 +21,7 @@
                     </state_interface>
                     <state_interface name="pos_fb">
+                        <param name="initial_value">0.0</param>
+                    </state_interface>
+                    <state_interface name="pos_cmd">
                         <param name="initial_value">0.0</param>
                     </state_interface>
@@ -58,4 +61,7 @@
                     <param name="initial_value">0.0</param>
                 </state_interface>
+                <state_interface name="pos_cmd">
+                    <param name="initial_value">0.0</param>
+                </state_interface>
                 <state_interface name="vel_fb">
                     <param name="initial_value">0.0</param>
@@ -74,4 +80,7 @@
                 </state_interface>
                 <state_interface name="pos_fb">
+                    <param name="initial_value">0.0</param>
+                </state_interface>
+                <state_interface name="pos_cmd">
                     <param name="initial_value">0.0</param>
                 </state_interface>
@@ -94,4 +103,7 @@
                     <param name="initial_value">0.0</param>
                 </state_interface>
+                <state_interface name="pos_cmd">
+                    <param name="initial_value">0.0</param>
+                </state_interface>
                 <state_interface name="vel_fb">
                     <param name="initial_value">0.0</param>
@@ -110,4 +122,7 @@
                 </state_interface>
                 <state_interface name="pos_fb">
+                    <param name="initial_value">0.0</param>
+                </state_interface>
+                <state_interface name="pos_cmd">
                     <param name="initial_value">0.0</param>
                 </state_interface>
@@ -130,4 +145,7 @@
                     <param name="initial_value">0.0</param>
                 </state_interface>
+                <state_interface name="pos_cmd">
+                    <param name="initial_value">0.0</param>
+                </state_interface>
                 <state_interface name="vel_fb">
                     <param name="initial_value">0.0</param>
@@ -148,4 +166,7 @@
                     <param name="initial_value">0.0</param>
                 </state_interface>
+                <state_interface name="pos_cmd">
+                    <param name="initial_value">0.0</param>
+                </state_interface>
                 <state_interface name="vel_fb">
                     <param name="initial_value">0.0</param>

Commit message: [WIP] estimated tool marker position

File: motoman_description/robots/hc10_macro.xacro (robot description, xacro)
@@ -149,5 +149,5 @@
     <link name="${prefix}tool_marker"/>
     <joint name="${prefix}tool0-marker" type="fixed">
-      <origin xyz="0 0 0.1" rpy="0 0 0"/>
+      <origin xyz="0 0 0.025" rpy="0 0 ${-pi/2}"/>
       <parent link="${prefix}tool0"/>
       <child link="${prefix}tool_marker"/>
