Commit message: fix urdf

File: motoman_description/robots/hc10dt_b10_macro.xacro (robot description, xacro)
@@ -7,5 +7,5 @@
       <visual>
         <geometry>
-          <mesh filename="package://motoman_hc10_support/meshes/hc10dt_b10/visual/base_link.dae"/>
+          <mesh filename="package://motoman_description/meshes/hc10dt_b10/visual/base_link.dae"/>
         </geometry>
         <xacro:material_yaskawa_blue/>
@@ -13,5 +13,5 @@
       <collision>
         <geometry>
-          <mesh filename="package://motoman_hc10_support/meshes/hc10dt_b10/collision/base_link.stl"/>
+          <mesh filename="package://motoman_description/meshes/hc10dt_b10/collision/base_link.stl"/>
         </geometry>
       </collision>
@@ -20,5 +20,5 @@
       <visual>
         <geometry>
-          <mesh filename="package://motoman_hc10_support/meshes/hc10dt_b10/visual/link_1_s.dae"/>
+          <mesh filename="package://motoman_description/meshes/hc10dt_b10/visual/link_1_s.dae"/>
         </geometry>
         <xacro:material_yaskawa_blue/>
@@ -26,5 +26,5 @@
       <collision>
         <geometry>
-          <mesh filename="package://motoman_hc10_support/meshes/hc10dt_b10/collision/link_1_s.stl"/>
+          <mesh filename="package://motoman_description/meshes/hc10dt_b10/collision/link_1_s.stl"/>
         </geometry>
       </collision>
@@ -33,5 +33,5 @@
       <visual>
         <geometry>
-          <mesh filename="package://motoman_hc10_support/meshes/hc10dt_b10/visual/link_2_l.dae"/>
+          <mesh filename="package://motoman_description/meshes/hc10dt_b10/visual/link_2_l.dae"/>
         </geometry>
         <xacro:material_yaskawa_blue/>
@@ -39,5 +39,5 @@
       <collision>
         <geometry>
-          <mesh filename="package://motoman_hc10_support/meshes/hc10dt_b10/collision/link_2_l.stl"/>
+          <mesh filename="package://motoman_description/meshes/hc10dt_b10/collision/link_2_l.stl"/>
         </geometry>
       </collision>
@@ -46,5 +46,5 @@
       <visual>
         <geometry>
-          <mesh filename="package://motoman_hc10_support/meshes/hc10dt_b10/visual/link_3_u.dae"/>
+          <mesh filename="package://motoman_description/meshes/hc10dt_b10/visual/link_3_u.dae"/>
         </geometry>
         <xacro:material_yaskawa_blue/>
@@ -52,5 +52,5 @@
       <collision>
         <geometry>
-          <mesh filename="package://motoman_hc10_support/meshes/hc10dt_b10/collision/link_3_u.stl"/>
+          <mesh filename="package://motoman_description/meshes/hc10dt_b10/collision/link_3_u.stl"/>
         </geometry>
       </collision>
@@ -59,5 +59,5 @@
       <visual>
         <geometry>
-          <mesh filename="package://motoman_hc10_support/meshes/hc10dt_b10/visual/link_4_r.dae"/>
+          <mesh filename="package://motoman_description/meshes/hc10dt_b10/visual/link_4_r.dae"/>
         </geometry>
         <xacro:material_yaskawa_blue/>
@@ -65,5 +65,5 @@
       <collision>
         <geometry>
-          <mesh filename="package://motoman_hc10_support/meshes/hc10dt_b10/collision/link_4_r.stl"/>
+          <mesh filename="package://motoman_description/meshes/hc10dt_b10/collision/link_4_r.stl"/>
         </geometry>
       </collision>
@@ -72,5 +72,5 @@
       <visual>
         <geometry>
-          <mesh filename="package://motoman_hc10_support/meshes/hc10dt_b10/visual/link_5_b.dae"/>
+          <mesh filename="package://motoman_description/meshes/hc10dt_b10/visual/link_5_b.dae"/>
         </geometry>
         <xacro:material_yaskawa_blue/>
@@ -78,5 +78,5 @@
       <collision>
         <geometry>
-          <mesh filename="package://motoman_hc10_support/meshes/hc10dt_b10/collision/link_5_b.stl"/>
+          <mesh filename="package://motoman_description/meshes/hc10dt_b10/collision/link_5_b.stl"/>
         </geometry>
       </collision>
@@ -85,5 +85,5 @@
       <visual>
         <geometry>
-          <mesh filename="package://motoman_hc10_support/meshes/hc10dt_b10/visual/link_6_t.dae"/>
+          <mesh filename="package://motoman_description/meshes/hc10dt_b10/visual/link_6_t.dae"/>
         </geometry>
         <xacro:material_yaskawa_blue/>
@@ -91,5 +91,5 @@
       <collision>
         <geometry>
-          <mesh filename="package://motoman_hc10_support/meshes/hc10dt_b10/collision/link_6_t.stl"/>
+          <mesh filename="package://motoman_description/meshes/hc10dt_b10/collision/link_6_t.stl"/>
        </geometry>
       </collision>

File: motoman_description/robots/hc10dt_macro.xacro (robot description, xacro)
@@ -7,5 +7,5 @@
       <visual>
         <geometry>
-          <mesh filename="package://motoman_hc10_support/meshes/hc10/visual/base_link.dae"/>
+          <mesh filename="package://motoman_description/meshes/hc10/visual/base_link.dae"/>
         </geometry>
         <xacro:material_yaskawa_blue/>
@@ -13,5 +13,5 @@
       <collision>
         <geometry>
-          <mesh filename="package://motoman_hc10_support/meshes/hc10/collision/base_link.stl"/>
+          <mesh filename="package://motoman_description/meshes/hc10/collision/base_link.stl"/>
         </geometry>
       </collision>
@@ -20,5 +20,5 @@
       <visual>
         <geometry>
-          <mesh filename="package://motoman_hc10_support/meshes/hc10/visual/link_1_s.dae"/>
+          <mesh filename="package://motoman_description/meshes/hc10/visual/link_1_s.dae"/>
         </geometry>
         <xacro:material_yaskawa_blue/>
@@ -26,5 +26,5 @@
       <collision>
         <geometry>
-          <mesh filename="package://motoman_hc10_support/meshes/hc10/collision/link_1_s.stl"/>
+          <mesh filename="package://motoman_description/meshes/hc10/collision/link_1_s.stl"/>
         </geometry>
       </collision>
@@ -33,5 +33,5 @@
       <visual>
         <geometry>
-          <mesh filename="package://motoman_hc10_support/meshes/hc10/visual/link_2_l.dae"/>
+          <mesh filename="package://motoman_description/meshes/hc10/visual/link_2_l.dae"/>
         </geometry>
         <xacro:material_yaskawa_blue/>
@@ -39,5 +39,5 @@
       <collision>
         <geometry>
-          <mesh filename="package://motoman_hc10_support/meshes/hc10/collision/link_2_l.stl"/>
+          <mesh filename="package://motoman_description/meshes/hc10/collision/link_2_l.stl"/>
         </geometry>
       </collision>
@@ -46,5 +46,5 @@
       <visual>
         <geometry>
-          <mesh filename="package://motoman_hc10_support/meshes/hc10/visual/link_3_u.dae"/>
+          <mesh filename="package://motoman_description/meshes/hc10/visual/link_3_u.dae"/>
         </geometry>
         <xacro:material_yaskawa_blue/>
@@ -52,5 +52,5 @@
       <collision>
         <geometry>
-          <mesh filename="package://motoman_hc10_support/meshes/hc10/collision/link_3_u.stl"/>
+          <mesh filename="package://motoman_description/meshes/hc10/collision/link_3_u.stl"/>
         </geometry>
       </collision>
@@ -59,5 +59,5 @@
       <visual>
         <geometry>
-          <mesh filename="package://motoman_hc10_support/meshes/hc10/visual/link_4_r.dae"/>
+          <mesh filename="package://motoman_description/meshes/hc10/visual/link_4_r.dae"/>
         </geometry>
         <xacro:material_yaskawa_blue/>
@@ -65,5 +65,5 @@
       <collision>
         <geometry>
-          <mesh filename="package://motoman_hc10_support/meshes/hc10/collision/link_4_r.stl"/>
+          <mesh filename="package://motoman_description/meshes/hc10/collision/link_4_r.stl"/>
         </geometry>
       </collision>
@@ -72,5 +72,5 @@
       <visual>
         <geometry>
-          <mesh filename="package://motoman_hc10_support/meshes/hc10/visual/link_5_b.dae"/>
+          <mesh filename="package://motoman_description/meshes/hc10/visual/link_5_b.dae"/>
         </geometry>
         <xacro:material_yaskawa_blue/>
@@ -78,5 +78,5 @@
       <collision>
         <geometry>
-          <mesh filename="package://motoman_hc10_support/meshes/hc10/collision/link_5_b.stl"/>
+          <mesh filename="package://motoman_description/meshes/hc10/collision/link_5_b.stl"/>
         </geometry>
       </collision>
@@ -85,5 +85,5 @@
       <visual>
         <geometry>
-          <mesh filename="package://motoman_hc10_support/meshes/hc10dt/visual/link_6_t.dae"/>
+          <mesh filename="package://motoman_description/meshes/hc10dt/visual/link_6_t.dae"/>
         </geometry>
         <xacro:material_yaskawa_blue/>
@@ -91,5 +91,5 @@
       <collision>
         <geometry>
-          <mesh filename="package://motoman_hc10_support/meshes/hc10dt/collision/link_6_t.stl"/>
+          <mesh filename="package://motoman_description/meshes/hc10dt/collision/link_6_t.stl"/>
        </geometry>
       </collision>

Commit message: fix hc10_dtp joint limits

File: motoman_description/robots/hc10dt_b10_macro.xacro (robot description, xacro)
@@ -102,5 +102,5 @@
       <origin xyz="0 0 0.275" rpy="0 0 0" />
       <axis xyz="0 0 1" />
-      <limit lower="${radians(-180)}" upper="${radians(180)}" effort="368.48" velocity="${radians(130)}"/>
+      <limit lower="${radians(-210)}" upper="${radians(210)}" effort="368.48" velocity="${radians(130)}"/>
     </joint>
     <joint name="${prefix}joint_2_l" type="revolute">
@@ -116,5 +116,5 @@
       <origin xyz="0 0 0.700" rpy="0 0 0" />
       <axis xyz="0 -1 0" />
-      <limit lower="${radians(-95)}" upper="${radians(265)}" effort="158.76" velocity="${radians(180)}"/>
+      <limit lower="${radians(-290)}" upper="${radians(290)}" effort="158.76" velocity="${radians(180)}"/>
     </joint>
     <joint name="${prefix}joint_4_r" type="revolute">
@@ -123,5 +123,5 @@
       <origin xyz="0.500 0 0" rpy="0 0 0" />
       <axis xyz="-1 0 0" />
-      <limit lower="${radians(-180)}" upper="${radians(180)}" effort="41.16" velocity="${radians(180)}"/>
+      <limit lower="${radians(-210)}" upper="${radians(210)}" effort="41.16" velocity="${radians(180)}"/>
     </joint>
     <joint name="${prefix}joint_5_b" type="revolute">
@@ -137,5 +137,5 @@
       <origin xyz="0 0 0" rpy="0 0 0" />
       <axis xyz="-1 0 0" />
-      <limit lower="${radians(-180)}" upper="${radians(180)}" effort="31.36" velocity="${radians(250)}"/>
+      <limit lower="${radians(-210)}" upper="${radians(210)}" effort="31.36" velocity="${radians(250)}"/>
     </joint>
     <!-- end of joint list -->

Commit message: basic gazebo support

File: motoman_description/robots/hc10dt_b10_macro.xacro (robot description, xacro)
@@ -5,4 +5,8 @@
     <!-- link list -->
     <link name="${prefix}base_link">
+      <inertial>
+        <mass value="1"/>
+        <inertia ixx="1"  ixy="0"  ixz="0" iyy="1" iyz="0" izz="1" />
+      </inertial>
       <visual>
         <geometry>
@@ -18,4 +22,8 @@
     </link>
     <link name="${prefix}link_1_s">
+      <inertial>
+        <mass value="1"/>
+        <inertia ixx="1"  ixy="0"  ixz="0" iyy="1" iyz="0" izz="1" />
+      </inertial>
       <visual>
         <geometry>
@@ -31,4 +39,8 @@
     </link>
     <link name="${prefix}link_2_l">
+      <inertial>
+        <mass value="1"/>
+        <inertia ixx="1"  ixy="0"  ixz="0" iyy="1" iyz="0" izz="1" />
+      </inertial>
       <visual>
         <geometry>
@@ -44,4 +56,8 @@
     </link>
     <link name="${prefix}link_3_u">
+      <inertial>
+        <mass value="1"/>
+        <inertia ixx="1"  ixy="0"  ixz="0" iyy="1" iyz="0" izz="1" />
+      </inertial>
       <visual>
         <geometry>
@@ -57,4 +73,8 @@
     </link>
     <link name="${prefix}link_4_r">
+      <inertial>
+        <mass value="1"/>
+        <inertia ixx="1"  ixy="0"  ixz="0" iyy="1" iyz="0" izz="1" />
+      </inertial>
       <visual>
         <geometry>
@@ -70,4 +90,8 @@
     </link>
     <link name="${prefix}link_5_b">
+      <inertial>
+        <mass value="1"/>
+        <inertia ixx="1"  ixy="0"  ixz="0" iyy="1" iyz="0" izz="1" />
+      </inertial>
       <visual>
         <geometry>
@@ -83,4 +107,8 @@
     </link>
     <link name="${prefix}link_6_t">
+      <inertial>
+        <mass value="1"/>
+        <inertia ixx="1"  ixy="0"  ixz="0" iyy="1" iyz="0" izz="1" />
+      </inertial>
       <visual>
         <geometry>

File: motoman_description/robots/ros2_control.xacro (robot description, xacro)
@@ -25,4 +25,7 @@
                     <plugin>mock_components/GenericSystem</plugin>
                 </xacro:if>
+                <xacro:if value="${sim_gazebo}">
+                    <plugin>gz_ros2_control/GazeboSimSystem</plugin>
+                </xacro:if>
                 <xacro:unless value="${use_mock_hardware or sim_gazebo}">
                     <plugin>motoman_hardware/MotomanHardware</plugin>
